File: Board Electronics/Board Electronics.sch (KiCad schematic (older format))
At the start: 9 parts, among them SW1 SW_SPDT_LED, U1 Powerboost1000C, U2 MCP23017, U3 MCP23017, U4 MCP23017, U6 Adafruit_Bluefruit_LE_UART_Fr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

Commit message: Finished Single Board PCB Design
Parts:
- added C1: C, Capacitors_THT:C_Disc_D6.0mm_W2.5mm_P5.00mm, symbol C
- added J1: CONN_01X06, Pin_Headers:Pin_Header_Straight_1x06_Pitch2.54mm, symbol CONN_01X06
- added J2: CONN_01X05, Pin_Headers:Pin_Header_Straight_1x05_Pitch2.54mm, symbol CONN_01X05
- added J3: CONN_02X12, Pin_Headers:Pin_Header_Straight_2x12_Pitch2.54mm, symbol CONN_02X12
- SW1: footprint (none) -> Pin_Headers:Pin_Header_Straight_1x05_Pitch2.54mm
- U1: renamed from U6; footprint (none) -> Extra-Parts:Blueferuit_LE_UART
- U2: renamed from U1; footprint (none) -> Extra-Parts:Powerboost1000c
- renumbered R122 to R2, R123 to R3, U2 to U3, U3 to U4, U4 to U5
Connections:
- net GND: now also SW1.1 (A), U2.7 (G), J1.1 (P1); no longer U2.10 (GOUT)
- net Route 1/A: now also U3.21 (GPA0); no longer U3.1 (GPB0)
- net Route 1/B: now also U3.22 (GPA1); no longer U3.2 (GPB1)
- net Route 1/C: now also U3.23 (GPA2); no longer U3.3 (GPB2)
- net Route 1/D: now also U3.24 (GPA3); no longer U3.4 (GPB3)
- net Route 1/E: now also U3.25 (GPA4); no longer U3.5 (GPB4)
- net Route 1/F: now also U3.26 (GPA5); no longer U3.6 (GPB5)
- net Route 1/G: now also U3.27 (GPA6); no longer U3.7 (GPB6)
- net Route 2/A: now also U3.1 (GPB0); no longer U3.21 (GPA0)
- net Route 2/B: now also U3.2 (GPB1); no longer U3.22 (GPA1)
- net Route 2/C: now also U3.3 (GPB2); no longer U3.23 (GPA2)
- net Route 2/D: now also U3.4 (GPB3); no longer U3.24 (GPA3)
- net Route 2/E: now also U3.5 (GPB4); no longer U3.25 (GPA4)
- net Route 2/F: now also U3.6 (GPB5); no longer U3.26 (GPA5)
- net Route 2/G: now also U3.7 (GPB6); no longer U3.27 (GPA6)
- net Route 3/A: now also U4.21 (GPA0); no longer U4.1 (GPB0)
- net Route 3/B: now also U4.22 (GPA1); no longer U4.2 (GPB1)
- net Route 3/C: now also U4.23 (GPA2); no longer U4.3 (GPB2)
- net Route 3/D: now also U4.24 (GPA3); no longer U4.4 (GPB3)
- net Route 3/E: now also U4.25 (GPA4); no longer U4.5 (GPB4)
- net Route 3/F: now also U4.26 (GPA5); no longer U4.6 (GPB5)
- net Route 3/G: now also U4.27 (GPA6); no longer U4.7 (GPB6)
- net Route 4/A: now also U4.1 (GPB0); no longer U4.21 (GPA0)
- net Route 4/B: now also U4.2 (GPB1); no longer U4.22 (GPA1)
- net Route 4/C: now also U4.3 (GPB2); no longer U4.23 (GPA2)
- net Route 4/D: now also U4.4 (GPB3); no longer U4.24 (GPA3)
- net Route 4/E: now also U4.5 (GPB4); no longer U4.25 (GPA4)
- net Route 4/F: now also U4.6 (GPB5); no longer U4.26 (GPA5)
- net Route 4/G: now also U4.7 (GPB6); no longer U4.27 (GPA6)
- net Route 5/A: now also U5.21 (GPA0); no longer U5.1 (GPB0)
- net Route 5/B: now also U5.22 (GPA1); no longer U5.2 (GPB1)
- net Route 5/C: now also U5.23 (GPA2); no longer U5.3 (GPB2)
- net Route 5/D: now also U5.24 (GPA3); no longer U5.4 (GPB3)
- net Route 5/E: now also U5.25 (GPA4); no longer U5.5 (GPB4)
- net Route 5/F: now also U5.26 (GPA5); no longer U5.6 (GPB5)
- net Route 5/G: now also U5.27 (GPA6); no longer U5.7 (GPB6)
- net Route 6/A: now also U5.1 (GPB0); no longer U5.21 (GPA0)
- net Route 6/B: now also U5.2 (GPB1); no longer U5.22 (GPA1)
- net Route 6/C: now also U5.3 (GPB2); no longer U5.23 (GPA2)
- net Route 6/D: now also U5.4 (GPB3); no longer U5.24 (GPA3)
- net Route 6/E: now also U5.5 (GPB4); no longer U5.25 (GPA4)
- net Route 6/F: now also U5.6 (GPB5); no longer U5.26 (GPA5)
- net Route 6/G: now also U5.7 (GPB6); no longer U5.27 (GPA6)
- net SCL: now also J3.19 (P19)
- net SDA: now also J3.17 (P17)
- net VCC: now also U2.8 (5V), J1.3 (P3), J2.1 (P1); no longer U2.9 (VOUT)
- net controller.sch/A1: now also J3.9 (P9)
- net controller.sch/A2: now also J3.11 (P11)
- net controller.sch/A3: now also J3.13 (P13)
- net controller.sch/RESET: now also C1.1
- net at U2.1 (VBUS): now also J2.5 (P5)
- net at U2.2 (BAT): now also J2.4 (P4)
- net at U2.3 (VS): now also J2.3 (P3)
- net at U2.5 (GND): now also J2.2 (P2); no longer SW1.1 (A)
- net U3INTB: now reaches U3.19 (INTB)
- net U3INTB: now also J3.8 (P8)
- net U3INTA: now reaches U3.20 (INTA)
- net U3INTA: now also J3.6 (P6)
- net U3A7: now reaches U3.28 (GPA7)
- net U3A7: now also J3.2 (P2)
- net U3B7: now reaches U3.8 (GPB7)
- net U3B7: now also J3.4 (P4)
- net U4INTB: now reaches U4.19 (INTB)
- net U4INTB: now also J3.16 (P16)
- net U4INTA: now reaches U4.20 (INTA)
- net U4INTA: now also J3.14 (P14)
- net U4A7: now reaches U4.28 (GPA7)
- net U4A7: now also J3.10 (P10)
- net U4B7: now reaches U4.8 (GPB7)
- net U4B7: now also J3.12 (P12)
- net U5INTB: now reaches U5.19 (INTB)
- net U5INTB: now also J3.24 (P24)
- net U5INTA: now reaches U5.20 (INTA)
- net U5INTA: now also J3.22 (P22)
- net U5A7: now reaches U5.28 (GPA7)
- net U5A7: now also J3.18 (P18)
- net U5B7: now reaches U5.8 (GPB7)
- net U5B7: now also J3.20 (P20)
- net BLE_DFU: now reaches U1.8 (DFU)
- net BLE_DFU: now also J3.21 (P21)
- new net 13: J3.3 (P3)
- new net 7: J3.1 (P1)
- new net AREF: J3.23 (P23)
- new net INT0: J3.7 (P7)
- new net INT1: J3.5 (P5)
- new net RST: C1.2, J1.6 (P6), J3.15 (P15)
- new net RX: J1.4 (P4)
- new net TX: J1.5 (P5)
- no-connect marks 0 -> 3
Other:
- note added: "ATMEGA Serial Port"
- note added: "Extra Ports Breakout"
- note added: "Power Breakout"
- moved on the sheet: U1
