File: Board Electronics/BusLoopId.sch (KiCad schematic (older format))
At the start: 43 parts, among them Q2 PN2222A, Q3 PN2222A, Q4 PN2222A

Commit message: Finished Single Board PCB Design
Parts:
- renumbered Q3 to Q1, Q4 to Q2, Q2 to Q3, R8 to R10, R9 to R11, R10 to R12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
