File: Board Electronics/Controller.sch (KiCad schematic (older format))
At the start: 4 parts, among them U5 ATMEGA328P-PU, Y1 Crystal

Commit message: Finished Single Board PCB Design
Parts:
- renumbered C1 to C2, C2 to C3, U5 to U6
Changed lines of the file:
@@
 $EndDescr
 $Comp
-L ATMEGA328P-PU U5
+L ATMEGA328P-PU U6
 U 1 1 58ADD6C3
 P 5200 3350
-F 0 "U5" H 4450 4600 50  0000 L BNN
+F 0 "U6" H 4450 4600 50  0000 L BNN
 F 1 "ATMEGA328P-PU" H 5600 1950 50  0000 L BNN
 F 2 "Housings_DIP:DIP-28_W7.62mm_Socket" H 5200 3350 50  0001 C CIN
@@
 XTAL_GND
 $Comp
-L C_Small C1
+L C_Small C2
 U 1 1 58AE41CC
 P 7200 2750
-F 0 "C1" H 7210 2820 50  0000 L CNN
+F 0 "C2" H 7210 2820 50  0000 L CNN
 F 1 "C20p" H 7210 2670 50  0000 L CNN
 F 2 "Capacitors_THT:C_Disc_D6_P5" H 7200 2750 50  0001 C CNN
@@
 $EndComp
 $Comp
-L C_Small C2
+L C_Small C3
 U 1 1 58AE4207
 P 7200 3050
-F 0 "C2" H 7210 3120 50  0000 L CNN
+F 0 "C3" H 7210 3120 50  0000 L CNN
 F 1 "C20p" H 7210 2970 50  0000 L CNN
 F 2 "Capacitors_THT:C_Disc_D6_P5" H 7200 3050 50  0001 C CNN
