File: Board Electronics/Board Electronics.kicad_pcb (KiCad board)
At the start: 2 copper layers, 270 parts, among them Q10 PN2222A, Q11 PN2222A, Q12 PN2222A, Q13 PN2222A, Q14 PN2222A, Q15 PN2222A, Q16 PN2222A, Q17 PN2222A, Q18 PN2222A, Q19 PN2222A, Q2 PN2222A, Q3 PN2222A, Q4 PN2222A, Q5 PN2222A, Q6 PN2222A, Q7 PN2222A, Q8 PN2222A, Q9 PN2222A, SW1 SW_Push_LED, U1 Powerboost1000C, U2 MCP23017, U3 MCP23017, U4 MCP23017, U5 ATMEGA328P-PU, Y1 Crystal

Commit message: Finished Single Board PCB Design
Parts:
- added C1: C, Capacitors_THT:C_Disc_D6.0mm_W2.5mm_P5.00mm, F.Cu at (347.5, 88.9)
- added J1: CONN_01X06, Pin_Headers:Pin_Header_Straight_1x06_Pitch2.54mm, F.Cu at (360.2, 78.7)
- added J2: CONN_01X05, Pin_Headers:Pin_Header_Straight_1x05_Pitch2.54mm, F.Cu at (283.5, 229.1)
- added J3: CONN_02X12, Pin_Headers:Pin_Header_Straight_2x12_Pitch2.54mm, F.Cu at (321.6, 116.8)
- added U2: Powerboost1000C, Extra-Parts:Powerboost1000c, F.Cu at (260.5, 193.7)
- SW1: value SW_Push_LED -> SW_SPDT_LED; footprint Pin_Headers:Pin_Header_Straight_2x02_Pitch1.27mm -> Pin_Headers:Pin_Header_Straight_1x05_Pitch2.54mm
- U1: value Powerboost1000C -> Adafruit_Bluefruit_LE_UART_Friend; footprint Housings_DIP:DIP-28_W7.62mm_Socket -> Extra-Parts:Blueferuit_LE_UART
- moved R3 202.2 mm to (341.9, 93.5), turned to 180 degrees
- moved R2 184.8 mm to (341.9, 87.4), turned to 180 degrees
- moved U6 130.6 mm to (352.2, 92.7)
- moved C2 130.6 mm to (337.8, 111.1)
- moved C3 130.6 mm to (337.8, 114.9)
- moved Y1 130.6 mm to (345.4, 110.6)
- moved R1 76.9 mm to (309.2, 226.7), turned to 180 degrees
- moved SW1 40.3 mm to (328.2, 217.4)
- moved U5 34.2 mm to (137.2, 191.8), turned to 0 degrees
- moved U3 33.9 mm to (138.4, 87.6), turned to 0 degrees
- moved U4 33.1 mm to (270.5, 120.7), turned to 180 degrees
- moved U1 17.5 mm to (364.5, 140.7), turned to 270 degrees
- moved Q10 1.98 mm to (203.2, 123.2)
- moved Q16 1.98 mm to (205.7, 182.1)
- renumbered C1 to C2, C2 to C3, Q3 to Q1, Q12 to Q10, Q13 to Q11, Q11 to Q12, Q15 to Q13, Q16 to Q14, Q14 to Q15, Q18 to Q16, Q19 to Q17, Q17 to Q18, Q4 to Q2, Q2 to Q3, Q6 to Q4, Q7 to Q5, Q5 to Q6, Q9 to Q7, Q10 to Q8, Q8 to Q9, R8 to R10, R98 to R100, R99 to R101, R100 to R102, R101 to R103, R102 to R104, R103 to R105, R104 to R106, R105 to R107, R106 to R108, R107 to R109, R9 to R11, R108 to R110, R109 to R111, R110 to R112, R111 to R113, R112 to R114, R113 to R115, R114 to R116, R115 to R117, R116 to R118, R117 to R119, R10 to R12, R118 to R120, R119 to R121, R120 to R122, R121 to R123, R11 to R13, R12 to R14, R13 to R15, R14 to R16, R15 to R17, R16 to R18, R17 to R19, R122 to R2, R18 to R20, R19 to R21, R20 to R22, R21 to R23, R22 to R24, R23 to R25, R24 to R26, R25 to R27, R26 to R28, R27 to R29, R123 to R3, R28 to R30, R29 to R31, R30 to R32, R31 to R33, R32 to R34, R33 to R35, R34 to R36, R35 to R37, R36 to R38, R37 to R39, R2 to R4, R38 to R40, R39 to R41, R40 to R42, R41 to R43, R42 to R44, R43 to R45, R44 to R46, R45 to R47, R46 to R48, R47 to R49, R3 to R5, R48 to R50, R49 to R51, R50 to R52, R51 to R53, R52 to R54, R53 to R55, R54 to R56, R55 to R57, R56 to R58, R57 to R59, R4 to R6, R58 to R60, R59 to R61, R60 to R62, R61 to R63, R62 to R64, R63 to R65, R64 to R66, R65 to R67, R66 to R68, R67 to R69, R5 to R7, R68 to R70, R69 to R71, R70 to R72, R71 to R73, R72 to R74, R73 to R75, R74 to R76, R75 to R77, R76 to R78, R77 to R79, R6 to R8, R78 to R80, R79 to R81, R80 to R82, R81 to R83, R82 to R84, R83 to R85, R84 to R86, R85 to R87, R86 to R88, R87 to R89, R7 to R9, R88 to R90, R89 to R91, R90 to R92, R91 to R93, R92 to R94, R93 to R95, R94 to R96, R95 to R97, R96 to R98, R97 to R99, U2 to U3, U3 to U4, U4 to U5, U5 to U6
Connections:
- SW1 pad 1: Net-(SW1-Pad1) -> /GND
- SW1 pad 3: /GND -> /controller.sch/A0
- U1 pad 1: Net-(U1-Pad1) -> /MOD
- U1 pad 2: Net-(U1-Pad2) -> /CTS
- U1 pad 3: Net-(U1-Pad3) -> /TXO
- U1 pad 4: Net-(SW1-Pad2) -> /RXI
- U1 pad 5: Net-(SW1-Pad1) -> /VCC
- U1 pad 6: /controller.sch/2/INT0 -> /RTS
- U1 pad 7: Net-(U1-Pad7) -> /GND
- U1 pad 8: Net-(U1-Pad8) -> /BLE_DFU
- U3 pad 1: /Route 1/A -> /Route 2/A
- U3 pad 19: Net-(U2-Pad19) -> /U3INTB
- U3 pad 2: /Route 1/B -> /Route 2/B
- U3 pad 20: Net-(U2-Pad20) -> /U3INTA
- U3 pad 21: /Route 2/A -> /Route 1/A
- U3 pad 22: /Route 2/B -> /Route 1/B
- U3 pad 23: /Route 2/C -> /Route 1/C
- U3 pad 24: /Route 2/D -> /Route 1/D
- U3 pad 25: /Route 2/E -> /Route 1/E
- U3 pad 26: /Route 2/F -> /Route 1/F
- U3 pad 27: /Route 2/G -> /Route 1/G
- U3 pad 28: Net-(U2-Pad28) -> /U3A7
- U3 pad 3: /Route 1/C -> /Route 2/C
- U3 pad 4: /Route 1/D -> /Route 2/D
- U3 pad 5: /Route 1/E -> /Route 2/E
- U3 pad 6: /Route 1/F -> /Route 2/F
- U3 pad 7: /Route 1/G -> /Route 2/G
- U3 pad 8: Net-(U2-Pad8) -> /U3B7
- U4 pad 1: /Route 3/A -> /Route 4/A
- U4 pad 19: Net-(U3-Pad19) -> /U4INTB
- U4 pad 2: /Route 3/B -> /Route 4/B
- U4 pad 20: Net-(U3-Pad20) -> /U4INTA
- U4 pad 21: /Route 4/A -> /Route 3/A
- U4 pad 22: /Route 4/B -> /Route 3/B
- U4 pad 23: /Route 4/C -> /Route 3/C
- U4 pad 24: /Route 4/D -> /Route 3/D
- U4 pad 25: /Route 4/E -> /Route 3/E
- U4 pad 26: /Route 4/F -> /Route 3/F
- U4 pad 27: /Route 4/G -> /Route 3/G
- U4 pad 28: Net-(U3-Pad28) -> /U4A7
- U4 pad 3: /Route 3/C -> /Route 4/C
- U4 pad 4: /Route 3/D -> /Route 4/D
- U4 pad 5: /Route 3/E -> /Route 4/E
- U4 pad 6: /Route 3/F -> /Route 4/F
- U4 pad 7: /Route 3/G -> /Route 4/G
- U4 pad 8: Net-(U3-Pad8) -> /U4B7
- U5 pad 1: /Route 5/A -> /Route 6/A
- U5 pad 19: Net-(U4-Pad19) -> /U5INTB
- U5 pad 2: /Route 5/B -> /Route 6/B
- U5 pad 20: Net-(U4-Pad20) -> /U5INTA
- U5 pad 21: /Route 6/A -> /Route 5/A
- U5 pad 22: /Route 6/B -> /Route 5/B
- U5 pad 23: /Route 6/C -> /Route 5/C
- U5 pad 24: /Route 6/D -> /Route 5/D
- U5 pad 25: /Route 6/E -> /Route 5/E
- U5 pad 26: /Route 6/F -> /Route 5/F
- U5 pad 27: /Route 6/G -> /Route 5/G
- U5 pad 28: Net-(U4-Pad28) -> /U5A7
- U5 pad 3: /Route 5/C -> /Route 6/C
- U5 pad 4: /Route 5/D -> /Route 6/D
- U5 pad 5: /Route 5/E -> /Route 6/E
- U5 pad 6: /Route 5/F -> /Route 6/F
- U5 pad 7: /Route 5/G -> /Route 6/G
- U5 pad 8: Net-(U4-Pad8) -> /U5B7
- U6 pad 13: /controller.sch/7 -> /7
- U6 pad 14: /controller.sch/8 -> /RTS
- U6 pad 15: /controller.sch/9 -> /RXI
- U6 pad 16: /controller.sch/10 -> /TXO
- U6 pad 17: /controller.sch/11 -> /CTS
- U6 pad 18: /controller.sch/12 -> /MOD
- U6 pad 19: /controller.sch/13 -> /13
- U6 pad 2: /controller.sch/0/RX -> /RX
- U6 pad 21: /controller.sch/AREF -> /AREF
- U6 pad 3: /controller.sch/1/TX -> /TX
- U6 pad 4: /controller.sch/2/INT0 -> /INT0
- U6 pad 5: /controller.sch/3/INT1 -> /INT1
Routing:
- net /CKA: track 88.9 -> 500.5 mm, vias 1 -> 4
- net /SDA: track 0.00 -> 366.0 mm, vias 0 -> 4
- net /SCL: track 0.00 -> 364.6 mm, vias 0 -> 3
- net /CKB: track 91.1 -> 452.0 mm, vias 1 -> 7
- net /CKC: track 90.5 -> 405.3 mm, vias 1 -> 5
- net /U5B7: track 0.00 -> 282.2 mm, vias 0 -> 1
- net /U5INTB: track 0.00 -> 274.8 mm, vias 0 -> 2
- net /U5INTA: track 0.00 -> 273.1 mm, vias 0 -> 1
- net /U5A7: track 0.00 -> 263.7 mm
- net /U3A7: track 0.00 -> 199.8 mm, vias 0 -> 3
- net /U3B7: track 0.00 -> 186.9 mm, vias 0 -> 2
- net /U3INTB: track 0.00 -> 184.3 mm, vias 0 -> 4
- net /controller.sch/A0: track 0.00 -> 179.4 mm
- net /U3INTA: track 0.00 -> 174.6 mm, vias 0 -> 2
- net /GND: track 0.70 -> 141.9 mm, vias 0 -> 7
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- added copper zone on F.Cu, net /GND
- added copper zone on B.Cu, net /VCC
Other:
- board outline added: 323.9 x 196.8 mm
- board text added: "13"
- board text added: "5V"
- board text added: "5V on Back"
- board text added: "7"
- board text added: "A1"
- board text added: "A2"
- board text added: "A3"
- board text added: "AREF"
- board text added: "ATMEGA UART"
- board text added: "BLE DFU"
- board text added: "Bat"
- board text added: "Common"
- board text added: "DTR"
- board text added: "Expansion Header"
- board text added: "GND"
- board text added: "INT0"
- board text added: "INT1"
- board text added: "LED GND"
- board text added: "LED VCC"
- board text added: "OFF"
- board text added: "ON"
- board text added: "Powerboost 1000C Extra Pins"
- board text added: "RESET"
- board text added: "RX"
- board text added: "SCL"
- board text added: "SDA"
- board text added: "TX"
- board text added: "U3 A7"
- board text added: "U3 B7"
- board text added: "U3 INT A"
- board text added: "U3 INT B"
- board text added: "U4 A7"
- board text added: "U4 B7"
- board text added: "U4 INT A"
- board text added: "U4 INT B"
- board text added: "U5 A7"
- board text added: "U5 B7"
- board text added: "U5 INT A"
- board text added: "U5 INT B"
- board text added: "USB"
- board text added: "VCC"
- board text added: "VS"

Commit message: added copper pours
Other:
- board text removed: "5V on Back"
Changed lines of the file:
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@@
   (general
     (links 483)
-    (no_connects 0)
+    (no_connects 48)
     (area 57.074999 38.024999 381.075001 235.025001)
     (thickness 1.6)
-    (drawings 65)
+    (drawings 64)
     (tracks 1635)
     (zones 0)
@@
   (page A3)
   (layers
-    (0 F.Cu mixed hide)
-    (31 B.Cu mixed hide)
+    (0 F.Cu mixed)
+    (31 B.Cu mixed)
     (33 F.Adhes user)
     (34 B.Paste user)
@@
     (effects (font (size 1.5 1.5) (thickness 0.3)))
   )
-  (gr_text "5V on Back" (at 258.572 245.364) (layer F.Cu)
-    (effects (font (size 12.7 12.7) (thickness 3.175)))
-  )
   (gr_line (start 381 38.1) (end 57.15 38.1) (layer Edge.Cuts) (width 0.15))
   (gr_line (start 381 38.1) (end 381 234.95) (layer Edge.Cuts) (width 0.15))
@@
     (connect_pads (clearance 0.508))
     (min_thickness 0.254)
-    (fill (arc_segments 16) (thermal_gap 0.508) (thermal_bridge_width 0.889))
+    (fill yes (arc_segments 16) (thermal_gap 0.508) (thermal_bridge_width 0.889))
     (polygon
       (pts
@@
     (connect_pads (clearance 0.508))
     (min_thickness 0.254)
-    (fill (arc_segments 16) (thermal_gap 0.508) (thermal_bridge_width 0.889))
+    (fill yes (arc_segments 16) (thermal_gap 0.508) (thermal_bridge_width 0.889))
     (polygon
       (pts

Commit message: update Kicad files to have new schematic design
This new schematic design is nested under a new folder called
alternative board electronics. It breaks apart the control circuitry and
the led attachment points to save PCB space (and this cost).

This may become the default schematics in a future revision, and the
all-in-one board will become the alternative.
Parts:
- added REF**: MountingHole_5.5mm, Mounting_Holes:MountingHole_5.5mm, F.Cu at (64.1, 45.1)
- added REF**: MountingHole_5.5mm, Mounting_Holes:MountingHole_5.5mm, F.Cu at (67.3, 224.8)
- R1, R10, R100, R101, R102, R103, R104, R105, R106, R107, R108, R109, R11, R110, R111, R112, R113, R114, R115, R116, R117, R118, R119, R12, R120, R121, R122, R123, R13, R14, R15, R16, R17, R18, R19, R2, R20, R21, R22, R23, R24, R25, R26, R27, R28, R29, R3, R30, R31, R32, R33, R34, R35, R36, R37, R38, R39, R4, R40, R41, R42, R43, R44, R45, R46, R47, R48, R49, R5, R50, R51, R52, R53, R54, R55, R56, R57, R58, R59, R6, R60, R61, R62, R63, R64, R65, R66, R67, R68, R69, R7, R70, R71, R72, R73, R74, R75, R76, R77, R78, R79, R8, R80, R81, R82, R83, R84, R85, R86, R87, R88, R89, R9, R90, R91, R92, R93, R94, R95, R96, R97, R98, R99: footprint Resistors_ThroughHole:R_Axial_DIN0309_L9.0mm_D3.2mm_P12.70mm_Horizontal -> Resistors_THT:R_Axial_DIN0309_L9.0mm_D3.2mm_P12.70mm_Horizontal
Connections:
- J1 pad 2: Net-(J1-Pad2) -> (no net)
- U2 pad 10: Net-(U2-Pad10) -> (no net)
- U2 pad 9: Net-(U2-Pad9) -> (no net)
Other:
- board size 323.9 x 196.8 mm -> 323.9 x 196.9 mm
