File: Board-electronics/Control Board/Board Electronics - Copy.kicad_pcb (KiCad board)
At the start: 2 copper layers, 135.9 x 81.3 mm, 31 parts, among them J1 CONN_01X06, J2 CONN_01X06, J3 CONN_02X12, J4 CONN_02X06, J5 CONN_02X06, J6 CONN_02X06, J7 CONN_02X06, J8 CONN_02X06, J9 CONN_02X06, M4 MountingHole_4.3mm_M4_Pad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

Commit message: more tweaking for perfection
Parts:
- added J10: CONN_02X01, Pin_Headers:Pin_Header_Straight_2x01_Pitch2.54mm, F.Cu at (195.3, 113.3)
- added R4: R, Resistors_THT:R_Axial_DIN0309_L9.0mm_D3.2mm_P12.70mm_Horizontal, F.Cu at (192.5, 106.9)
Routing:
- net (no net): track 13.7 -> 0.00 mm, vias 1 -> 0
- net Net-(J10-Pad1): track 0.00 -> 8.09 mm
- net /CKA: track 278.8 -> 271.3 mm
- net /controller.sch/A0: track 129.1 -> 127.4 mm
- net /SCL: track 191.4 -> 192.6 mm
- net /RX: track 26.2 -> 25.1 mm
- net /GND: track 65.5 -> 64.5 mm
- net /SDA: track 195.1 -> 196.0 mm
- net Net-(J8-Pad8): track 9.01 -> 8.25 mm
- net Net-(J8-Pad10): track 9.01 -> 8.25 mm
- net Net-(J8-Pad6): track 9.01 -> 8.25 mm
- net Net-(J8-Pad4): track 9.01 -> 8.25 mm
- net /TX: track 28.7 -> 28.1 mm
