File: Board-electronics/Control Board/Board Electronics.sch (KiCad schematic (older format))
At the start: 20 parts, among them J1 CONN_01X06, J10 CONN_02X01, J2 CONN_01X06, J3 CONN_02X12, J4 CONN_02X06, J5 CONN_02X06, J6 CONN_02X06, J7 CONN_02X06, J8 CONN_02X06, J9 CONN_02X06, SW1 SW_SPDT_LED, U1 Adafruit_Bluefruit_LE_UART_Fr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, U2 Powerboost1000C, U3 MCP23017, U4 MCP23017, U5 MCP23017

Commit message: more tweaking for perfection
Parts:
- added R4: R, Resistors_THT:R_Axial_DIN0207_L6.3mm_D2.5mm_P10.16mm_Horizontal, symbol R
- J10: footprint (none) -> Pin_Headers:Pin_Header_Straight_2x01_Pitch2.54mm
- R1, R2, R3: footprint Resistors_THT:R_Axial_DIN0309_L9.0mm_D3.2mm_P12.70mm_Horizontal -> Resistors_THT:R_Axial_DIN0207_L6.3mm_D2.5mm_P10.16mm_Horizontal
Connections:
- net GND: no longer U5.16 (A1)
- net VCC: now also U5.16 (A1), R4.2; no longer J10.1 (P1)
- new net: J10.1 (P1), R4.1
Other:
- moved on the sheet: J10
Changed lines of the file:
@@
 VCC
 Text Label 7050 9000 0    60   ~ 0
-GND
+VCC
 Text Label 7050 9100 0    60   ~ 0
 GND
@@
 F 0 "R1" V 3280 2850 50  0000 C CNN
 F 1 "R220" V 3200 2850 50  0000 C CNN
-F 2 "Resistors_THT:R_Axial_DIN0309_L9.0mm_D3.2mm_P12.70mm_Horizontal" V 3130 2850 50  0001 C CNN
+F 2 "Resistors_THT:R_Axial_DIN0207_L6.3mm_D2.5mm_P10.16mm_Horizontal" V 3130 2850 50  0001 C CNN
 F 3 "" H 3200 2850 50  0001 C CNN
 	1    3200 2850
@@
 F 0 "R2" V 4030 5600 50  0000 C CNN
 F 1 "R4K7" V 3950 5600 50  0000 C CNN
-F 2 "Resistors_THT:R_Axial_DIN0309_L9.0mm_D3.2mm_P12.70mm_Horizontal" V 3880 5600 50  0001 C CNN
+F 2 "Resistors_THT:R_Axial_DIN0207_L6.3mm_D2.5mm_P10.16mm_Horizontal" V 3880 5600 50  0001 C CNN
 F 3 "" H 3950 5600 50  0001 C CNN
 	1    3950 5600
@@
 F 0 "R3" V 4180 5600 50  0000 C CNN
 F 1 "R4K7" V 4100 5600 50  0000 C CNN
-F 2 "Resistors_THT:R_Axial_DIN0309_L9.0mm_D3.2mm_P12.70mm_Horizontal" V 4030 5600 50  0001 C CNN
+F 2 "Resistors_THT:R_Axial_DIN0207_L6.3mm_D2.5mm_P10.16mm_Horizontal" V 4030 5600 50  0001 C CNN
 F 3 "" H 4100 5600 50  0001 C CNN
 	1    4100 5600
@@
 L CONN_02X01 J10
 U 1 1 59133179
-P 5950 2050
-F 0 "J10" H 5950 2150 50  0000 C CNN
-F 1 "CONN_02X01" H 5950 1950 50  0000 C CNN
-F 2 "" H 5950 850 50  0001 C CNN
-F 3 "" H 5950 850 50  0001 C CNN
-	1    5950 2050
+P 6250 2400
+F 0 "J10" H 6250 2500 50  0000 C CNN
+F 1 "CONN_02X01" H 6250 2300 50  0000 C CNN
+F 2 "Pin_Headers:Pin_Header_Straight_2x01_Pitch2.54mm" H 6250 1200 50  0001 C CNN
+F 3 "" H 6250 1200 50  0001 C CNN
+	1    6250 2400
 	1    0    0    -1
 $EndComp
-Text Label 5700 2050 2    60   ~ 0
-VCC
-Text Label 6200 2050 0    60   ~ 0
-GND
+Text Label 6500 2400 0    60   ~ 0
+GND
+$Comp
+L R R4
+U 1 1 5913FDF5
+P 5800 2400
+F 0 "R4" V 5880 2400 50  0000 C CNN
+F 1 "R" V 5800 2400 50  0000 C CNN
+F 2 "Resistors_THT:R_Axial_DIN0207_L6.3mm_D2.5mm_P10.16mm_Horizontal" V 5730 2400 50  0001 C CNN
+F 3 "" H 5800 2400 50  0001 C CNN
+	1    5800 2400
+	0    1    1    0
+$EndComp
+Wire Wire Line
+	5950 2400 6000 2400
+Text Label 5550 2400 2    60   ~ 0
+VCC
+Wire Wire Line
+	5550 2400 5650 2400
 $EndSCHEMATC

Commit message: just some more tweaks
Parts:
- removed J3: CONN_02X12, Pin_Headers:Pin_Header_Straight_2x12_Pitch2.54mm, symbol CONN_02X12
- added C2, C3, C4: C.1u, Capacitors_THT:C_Disc_D6.0mm_W4.4mm_P5.00mm, symbol C
- added J3: CONN_01X12, Pin_Headers:Pin_Header_Straight_1x12_Pitch2.54mm, symbol CONN_01X12
- added R1: R4.7K, Resistors_THT:R_Axial_DIN0207_L6.3mm_D2.5mm_P10.16mm_Horizontal, symbol R
- C1: footprint Capacitors_THT:C_Disc_D6.0mm_W2.5mm_P5.00mm -> Capacitors_THT:C_Disc_D6.0mm_W4.4mm_P5.00mm
- U3, U4, U5: footprint Housings_DIP:DIP-28_W7.62mm_Socket -> Housings_DIP:DIP-28_W7.62mm_LongPads
- renumbered J9 to J10, J10 to J4, J4 to J5, J5 to J6, J6 to J7, J7 to J8, J8 to J9, R1 to R2, R2 to R3, R3 to R4, R4 to R5
Connections:
- net 13: now also J3.1 (P1)
- net 7: now also J3.2 (P2)
- net AREF: now also J3.9 (P9)
- net BLE_DFU: now also J3.12 (P12)
- net GND: now also C2.1, C3.1, C4.1
- net INT0: now also J3.4 (P4)
- net INT1: now also J3.3 (P3)
- net RST: now also C1.1, J3.8 (P8); no longer C1.2
- net SCL: now also J3.10 (P10)
- net SDA: now also J3.11 (P11)
- net VCC: now also C2.2, C3.2, C4.2, R1.2
- net controller.sch/RESET: now also C1.2, R1.1; no longer C1.1
- net VBUS: now reaches J2.5 (P5), U2.1 (VBUS)
- net BAT: now reaches J2.4 (P4), U2.2 (BAT)
- net VS: now reaches J2.3 (P3), U2.3 (VS)
- net SW1_COM: now reaches SW1.2 (B), U2.4 (EN)
- net G: now reaches J2.2 (P2), J2.6 (P6), U2.5 (GND)
- net at U3.27 (GPA6): now also J6.11 (P11); no longer J6.9 (P9)
- net at U3.7 (GPB6): now also J5.11 (P11); no longer J5.9 (P9)
- net at U4.27 (GPA6): now also J8.11 (P11); no longer J8.9 (P9)
- net at U4.7 (GPB6): now also J7.11 (P11); no longer J7.9 (P9)
- net at U5.27 (GPA6): now also J10.11 (P11); no longer J10.9 (P9)
- net at U5.7 (GPB6): now also J9.11 (P11); no longer J9.9 (P9)
- net U3A7: no longer names the net of U3.28 (GPA7)
- net U3B7: no longer names the net of U3.8 (GPB7)
- net U3INTA: no longer names the net of U3.20 (INTA)
- net U3INTB: no longer names the net of U3.19 (INTB)
- net U4A7: no longer names the net of U4.28 (GPA7)
- net U4B7: no longer names the net of U4.8 (GPB7)
- net U4INTA: no longer names the net of U4.20 (INTA)
- net U4INTB: no longer names the net of U4.19 (INTB)
- net U5A7: no longer names the net of U5.28 (GPA7)
- net U5B7: no longer names the net of U5.8 (GPB7)
- net U5INTA: no longer names the net of U5.20 (INTA)
- net U5INTB: no longer names the net of U5.19 (INTB)
- net controller.sch/A0 renamed A0
- new net A1: J3.5 (P5)
- new net A2: J3.6 (P6)
- new net A3: J3.7 (P7)
- no-connect marks 9 -> 21
Other:
- moved on the sheet: C1
