File: Board-electronics/Control Board/Controller.sch (KiCad schematic (older format))
At the start: 4 parts, among them U6 ATMEGA328P-PU, Y1 Crystal

Commit message: just some more tweaks
Parts:
- added C5: C10u, Capacitors_THT:C_Disc_D6.0mm_W4.4mm_P5.00mm, symbol C
- added C6, C7: C.1u, Capacitors_THT:C_Disc_D6.0mm_W4.4mm_P5.00mm, symbol C
- added C8: C4.7u, Capacitors_THT:C_Disc_D7.5mm_W5.0mm_P5.00mm, symbol C
- U6: footprint Housings_DIP:DIP-28_W7.62mm_Socket -> Housings_DIP:DIP-28_W7.62mm_LongPads
- renumbered C3 to C10, C2 to C9
Connections:
- net GND: now also C5.2, C6.1, C7.2, C8.1
- net VCC: now also C5.1, C6.2, C7.1, C8.2
Changed lines of the file:
@@
 encoding utf-8
 Sheet 2 2
-Title ""
-Date ""
-Rev ""
+Title "Control Board ATMEGA setup"
+Date "2017-05-16"
+Rev "1"
 Comp ""
 Comment1 ""
@@
 F 0 "U6" H 4450 4600 50  0000 L BNN
 F 1 "ATMEGA328P-PU" H 5600 1950 50  0000 L BNN
-F 2 "Housings_DIP:DIP-28_W7.62mm_Socket" H 5200 3350 50  0001 C CIN
+F 2 "Housings_DIP:DIP-28_W7.62mm_LongPads" H 5200 3350 50  0001 C CIN
 F 3 "" H 5200 3350 50  0001 C CNN
 	1    5200 3350
@@
 Text HLabel 4000 4500 0    60   Input ~ 0
 GND
-Wire Wire Line
-	4000 4500 4100 4500
-Wire Wire Line
-	4100 4450 4100 4800
-Wire Wire Line
-	4100 4550 4300 4550
-Wire Wire Line
-	4100 4450 4300 4450
-Connection ~ 4100 4500
-Text HLabel 3700 2400 0    60   Input ~ 0
+Text HLabel 2950 2450 0    60   Input ~ 0
 VCC
-Wire Wire Line
-	3700 2400 3950 2400
-Wire Wire Line
-	3950 2250 3950 2550
-Wire Wire Line
-	3950 2250 4300 2250
-Wire Wire Line
-	3950 2550 4300 2550
-Connection ~ 3950 2400
-Connection ~ 4100 4550
 Text Label 4100 4800 2    60   ~ 0
 XTAL_GND
-Wire Wire Line
-	7550 2900 7850 2900
 Text Label 7850 2900 0    60   ~ 0
 XTAL_GND
 $Comp
-L C_Small C2
+L C_Small C9
 U 1 1 58AE41CC
 P 7200 2750
-F 0 "C2" H 7210 2820 50  0000 L CNN
+F 0 "C9" H 7210 2820 50  0000 L CNN
 F 1 "C20p" H 7210 2670 50  0000 L CNN
 F 2 "Capacitors_THT:C_Disc_D6.0mm_W2.5mm_P5.00mm" H 7200 2750 50  0001 C CNN
@@
 $EndComp
 $Comp
-L C_Small C3
+L C_Small C10
 U 1 1 58AE4207
 P 7200 3050
-F 0 "C3" H 7210 3120 50  0000 L CNN
+F 0 "C10" H 7210 3120 50  0000 L CNN
 F 1 "C20p" H 7210 2970 50  0000 L CNN
 F 2 "Capacitors_THT:C_Disc_D6.0mm_W2.5mm_P5.00mm" H 7200 3050 50  0001 C CNN
@@
 	0    1    1    0
 $EndComp
-Wire Wire Line
-	6200 2850 6600 2850
-Wire Wire Line
-	6600 2850 6600 2750
-Wire Wire Line
-	6600 2750 7100 2750
-Wire Wire Line
-	6600 2950 6600 3050
-Wire Wire Line
-	6600 3050 7100 3050
-Connection ~ 6850 3050
-Connection ~ 6850 2750
-Wire Wire Line
-	7300 2750 7550 2750
-Wire Wire Line
-	7550 2750 7550 3050
-Wire Wire Line
-	7550 3050 7300 3050
-Connection ~ 7550 2900
-Wire Wire Line
-	6200 3850 6350 3850
-Wire Wire Line
-	6200 3950 6350 3950
-Wire Wire Line
-	6200 4050 6350 4050
-Wire Wire Line
-	6200 4150 6350 4150
-Wire Wire Line
-	6200 4250 6350 4250
-Wire Wire Line
-	6200 4350 6350 4350
-Wire Wire Line
-	6200 4450 6350 4450
-Wire Wire Line
-	6200 4550 6350 4550
-Wire Wire Line
-	6200 3100 6350 3100
-Wire Wire Line
-	6200 3200 6350 3200
-Wire Wire Line
-	6200 3300 6350 3300
-Wire Wire Line
-	6200 3400 6350 3400
-Wire Wire Line
-	6200 3500 6350 3500
-Wire Wire Line
-	6200 3600 6350 3600
-Wire Wire Line
-	6200 3700 6350 3700
-Wire Wire Line
-	6200 2350 6350 2350
-Wire Wire Line
-	6200 2450 6350 2450
-Wire Wire Line
-	6200 2550 6350 2550
-Wire Wire Line
-	6200 2650 6350 2650
-Wire Wire Line
-	6200 2750 6350 2750
-Wire Wire Line
-	4300 2850 4150 2850
-Wire Wire Line
-	6200 2950 6600 2950
 Text HLabel 6350 2250 2    60   Input ~ 0
 8
@@
 Text HLabel 4150 2850 0    60   Input ~ 0
 AREF
+$Comp
+L C C8
+U 1 1 591B7FA4
+P 3600 2100
+F 0 "C8" H 3625 2200 50  0000 L CNN
+F 1 "C4.7u" H 3625 2000 50  0000 L CNN
+F 2 "Capacitors_THT:C_Disc_D7.5mm_W5.0mm_P5.00mm" H 3638 1950 50  0001 C CNN
+F 3 "" H 3600 2100 50  0001 C CNN
+	1    3600 2100
+	1    0    0    -1
+$EndComp
+$Comp
+L C C6
+U 1 1 591B7FF2
+P 3350 2100
+F 0 "C6" H 3375 2200 50  0000 L CNN
+F 1 "C.1u" H 3375 2000 50  0000 L CNN
+F 2 "Capacitors_THT:C_Disc_D6.0mm_W4.4mm_P5.00mm" H 3388 1950 50  0001 C CNN
+F 3 "" H 3350 2100 50  0001 C CNN
+	1    3350 2100
+	1    0    0    -1
+$EndComp
+$Comp
+L C C7
+U 1 1 591B8155
+P 3550 2700
+F 0 "C7" H 3575 2800 50  0000 L CNN
+F 1 "C.1u" H 3575 2600 50  0000 L CNN
+F 2 "Capacitors_THT:C_Disc_D6.0mm_W4.4mm_P5.00mm" H 3588 2550 50  0001 C CNN
+F 3 "" H 3550 2700 50  0001 C CNN
+	1    3550 2700
+	1    0    0    -1
+$EndComp
+$Comp
+L C C5
+U 1 1 591B815B
+P 3300 2700
+F 0 "C5" H 3325 2800 50  0000 L CNN
+F 1 "C10u" H 3325 2600 50  0000 L CNN
+F 2 "Capacitors_THT:C_Disc_D6.0mm_W4.4mm_P5.00mm" H 3338 2550 50  0001 C CNN
+F 3 "" H 3300 2700 50  0001 C CNN
+	1    3300 2700
+	1    0    0    -1
+$EndComp
+Wire Wire Line
+	4000 4500 4100 4500
+Wire Wire Line
+	4100 4450 4100 4800
+Wire Wire Line
+	4100 4550 4300 4550
+Wire Wire Line
+	4100 4450 4300 4450
+Connection ~ 4100 4500
+Wire Wire Line
+	2950 2450 3200 2450
+Connection ~ 3200 2450
+Connection ~ 4100 4550
+Wire Wire Line
+	7550 2900 7850 2900
+Wire Wire Line
+	6200 2850 6600 2850
+Wire Wire Line
+	6600 2850 6600 2750
+Wire Wire Line
+	6600 2750 7100 2750
+Wire Wire Line
+	6600 2950 6600 3050
+Wire Wire Line
+	6600 3050 7100 3050
+Connection ~ 6850 3050
+Connection ~ 6850 2750
+Wire Wire Line
+	7300 2750 7550 2750
+Wire Wire Line
+	7550 2750 7550 3050
+Wire Wire Line
+	7550 3050 7300 3050
+Connection ~ 7550 2900
+Wire Wire Line
+	6200 3850 6350 3850
+Wire Wire Line
+	6200 3950 6350 3950
+Wire Wire Line
+	6200 4050 6350 4050
+Wire Wire Line
+	6200 4150 6350 4150
+Wire Wire Line
+	6200 4250 6350 4250
+Wire Wire Line
+	6200 4350 6350 4350
+Wire Wire Line
+	6200 4450 6350 4450
+Wire Wire Line
+	6200 4550 6350 4550
+Wire Wire Line
+	6200 3100 6350 3100
+Wire Wire Line
+	6200 3200 6350 3200
+Wire Wire Line
+	6200 3300 6350 3300
+Wire Wire Line
+	6200 3400 6350 3400
+Wire Wire Line
+	6200 3500 6350 3500
+Wire Wire Line
+	6200 3600 6350 3600
+Wire Wire Line
+	6200 3700 6350 3700
+Wire Wire Line
+	6200 2350 6350 2350
+Wire Wire Line
+	6200 2450 6350 2450
+Wire Wire Line
+	6200 2550 6350 2550
+Wire Wire Line
+	6200 2650 6350 2650
+Wire Wire Line
+	6200 2750 6350 2750
+Wire Wire Line
+	4300 2850 4150 2850
+Wire Wire Line
+	6200 2950 6600 2950
 Wire Wire Line
 	6200 2250 6350 2250
+Wire Wire Line
+	3200 2250 4300 2250
+Connection ~ 3600 2250
+Connection ~ 3350 2250
+Wire Wire Line
+	3200 2250 3200 2550
+Wire Wire Line
+	3200 2550 4300 2550
+Connection ~ 3300 2550
+Connection ~ 3550 2550
+Text Label 3600 1950 1    60   ~ 0
+GND
+Text Label 3350 1950 1    60   ~ 0
+GND
+Text Label 3300 2850 3    60   ~ 0
+GND
+Text Label 3550 2850 3    60   ~ 0
+GND
 $EndSCHEMATC
