File: Board-electronics/Control Board/Board Electronics.kicad_pcb (KiCad board)
At the start: 2 copper layers, 135.9 x 81.3 mm, 32 parts, among them J1 CONN_01X06, J10 CONN_02X01, J2 CONN_01X06, J3 CONN_02X12, J4 CONN_02X06, J5 CONN_02X06, J6 CONN_02X06, J7 CONN_02X06, J8 CONN_02X06, J9 CONN_02X06, M4 MountingHole_4.3mm_M4_Pad, SW1 SW_SPDT_LED, U1 Adafruit_Bluefruit_LE_UART_Fr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, U2 Powerboost1000C, U3 MCP23017, U4 MCP23017, U5 MCP23017, U6 ATMEGA328P-PU, Y1 Crystal

Commit message: more tweaking for perfection
Parts:
- added R4: R, Resistors_THT:R_Axial_DIN0207_L6.3mm_D2.5mm_P10.16mm_Horizontal, F.Cu at (203.1, 113.4)
- R1, R2, R3: footprint Resistors_THT:R_Axial_DIN0309_L9.0mm_D3.2mm_P12.70mm_Horizontal -> Resistors_THT:R_Axial_DIN0207_L6.3mm_D2.5mm_P10.16mm_Horizontal
- moved J10 61.3 mm to (203.1, 109.5), turned to 0 degrees
- moved R1 3.75 mm to (102.1, 128.8)
- moved R3 3.66 mm to (108.0, 128.5)
- moved R2 3.06 mm to (113.8, 127.8)
Connections:
- J10 pad 1: /VCC -> Net-(J10-Pad1)
- U5 pad 16: /GND -> /VCC
Routing:
- net /CKC: track 323.0 -> 281.5 mm
- net /VCC: track 25.7 -> 49.5 mm
- net /GND: track 64.5 -> 80.0 mm
- net /U4INTB: track 76.5 -> 64.4 mm
- net /AREF: track 76.6 -> 85.8 mm
- net /SDA: track 196.0 -> 200.1 mm, vias 4 -> 3
- net Net-(J10-Pad1): track 0.00 -> 3.94 mm
- net /CKA: track 271.3 -> 274.8 mm, vias 6 -> 5
- net /CKB: track 275.4 -> 278.2 mm, vias 6 -> 7
- net /U4INTA: track 83.8 -> 86.1 mm, vias 2 -> 3
- net Net-(J2-Pad2): track 19.6 -> 21.3 mm
- net /SCL: track 192.6 -> 191.5 mm
- net /RX: track 25.1 -> 24.1 mm
- net Net-(R1-Pad1): track 69.6 -> 68.6 mm
- net /TX: track 28.1 -> 27.3 mm
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Other:
- net class Default: clearance 0.1524 -> 0.508; trace_width 0.1524 -> 0.254
- rule trace_clearance: 0.1524 -> 0.508
- rule trace_min: 0.1524 -> 0.254

Commit message: just some more tweaks
Parts:
- removed the R4 at (203.1, 113.4)
- added C2: C.1u, Capacitors_THT:C_Disc_D6.0mm_W4.4mm_P5.00mm, F.Cu at (119.4, 88.9)
- added C3: C.1u, Capacitors_THT:C_Disc_D6.0mm_W4.4mm_P5.00mm, F.Cu at (156.8, 88.8)
- added C4: C.1u, Capacitors_THT:C_Disc_D6.0mm_W4.4mm_P5.00mm, F.Cu at (194.1, 85.4)
- added C5: C10u, Capacitors_THT:C_Disc_D6.0mm_W4.4mm_P5.00mm, F.Cu at (200.7, 124.5)
- added C6: C.1u, Capacitors_THT:C_Disc_D6.0mm_W4.4mm_P5.00mm, F.Cu at (105.9, 127.5)
- added C7: C.1u, Capacitors_THT:C_Disc_D6.0mm_W4.4mm_P5.00mm, F.Cu at (95.0, 148.8)
- added C8: C4.7u, Capacitors_THT:C_Disc_D7.5mm_W5.0mm_P5.00mm, F.Cu at (105.9, 132.3)
- added R1: R4.7K, Resistors_THT:R_Axial_DIN0207_L6.3mm_D2.5mm_P10.16mm_Horizontal, F.Cu at (119.4, 135.1)
- added R5: R, Resistors_THT:R_Axial_DIN0207_L6.3mm_D2.5mm_P10.16mm_Horizontal, F.Cu at (203.1, 113.4)
- added REF**: Symbol_CreativeCommons_SilkScreenTop_Type2_Big, Extra-Parts:Symbol_CreativeCommons_SilkScreenTop_Type2_Big, F.Cu at (154.9, 109.2)
- C1: footprint Capacitors_THT:C_Disc_D6.0mm_W2.5mm_P5.00mm -> Capacitors_THT:C_Disc_D6.0mm_W4.4mm_P5.00mm
- J3: value CONN_02X12 -> CONN_01X12; footprint Pin_Headers:Pin_Header_Straight_2x12_Pitch2.54mm -> Pin_Headers:Pin_Header_Straight_1x12_Pitch2.54mm
- U1: moved to F.Cu
- U3, U4, U5, U6: footprint Housings_DIP:DIP-28_W7.62mm_Socket -> Housings_DIP:DIP-28_W7.62mm_LongPads
- moved REF*** 74.6 mm to (113.9, 109.1)
- moved R2 69.2 mm to (169.9, 142.7)
- moved U2 37.1 mm to (173.2, 153.8), turned to 90 degrees
- moved SW1 27.6 mm to (163.3, 135.1), turned to 0 degrees
- moved U1 21.3 mm to (149.6, 116.3)
- moved REF*** 21.2 mm to (126.0, 152.3)
- moved J1 20.9 mm to (112.1, 129.4), turned to 90 degrees
- moved G*** 16.8 mm to (156.5, 152.1)
- moved J2 16.1 mm to (201.9, 130.8), turned to 0 degrees
- moved REF*** 9.17 mm to (181.7, 131.2)
- moved R3 8.89 mm to (112.3, 119.0), turned to 180 degrees
- moved R4 6.65 mm to (110.9, 122.6), turned to 180 degrees
- moved M4 5.08 mm to (203.2, 152.4)
- moved M4 5.08 mm to (203.2, 86.4)
- moved C1 4.44 mm to (124.5, 133.2)
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- renumbered C3 to C10, C2 to C9, J9 to J10, J10 to J4, J4 to J5, J5 to J6, J6 to J7, J7 to J8, J8 to J9, R1 to R2, R2 to R3, R3 to R4
Connections:
- net /controller.sch/A0 renamed /A0
- net Net-(J2-Pad2) renamed /G
- net Net-(J2-Pad3) renamed /VS
- net Net-(J2-Pad4) renamed /BAT
- net Net-(J2-Pad5) renamed /VBUS
- net Net-(SW1-Pad2) renamed /SW1_COM
- C1 pad 1: /controller.sch/RESET -> /RST
- C1 pad 2: /RST -> /controller.sch/RESET
- J10 pad 11: (no net) -> Net-(J10-Pad11)
- J10 pad 9: Net-(J9-Pad9) -> (no net)
- J3 pad 1: /U3A7 -> /13
- J3 pad 10: /controller.sch/A1 -> /SCL
- J3 pad 11: /U4B7 -> /SDA
- J3 pad 12: /controller.sch/A2 -> /BLE_DFU
- J3 pad 3: /U3B7 -> /INT1
- J3 pad 4: /13 -> /INT0
- J3 pad 5: /U3INTA -> /A1
- J3 pad 6: /INT1 -> /A2
- J3 pad 7: /U3INTB -> /A3
- J3 pad 8: /INT0 -> /RST
- J3 pad 9: /U4A7 -> /AREF
- J5 pad 11: (no net) -> Net-(J5-Pad11)
- J5 pad 9: Net-(J4-Pad9) -> (no net)
- J6 pad 11: (no net) -> Net-(J6-Pad11)
- J6 pad 9: Net-(J5-Pad9) -> (no net)
- J7 pad 11: (no net) -> Net-(J7-Pad11)
- J7 pad 9: Net-(J6-Pad9) -> (no net)
- J8 pad 11: (no net) -> Net-(J8-Pad11)
- J8 pad 9: Net-(J7-Pad9) -> (no net)
- J9 pad 11: (no net) -> Net-(J9-Pad11)
- J9 pad 9: Net-(J8-Pad9) -> (no net)
- U3 pad 19: /U3INTB -> (no net)
- U3 pad 20: /U3INTA -> (no net)
- U3 pad 27: Net-(J5-Pad9) -> Net-(J6-Pad11)
- U3 pad 28: /U3A7 -> (no net)
- U3 pad 7: Net-(J4-Pad9) -> Net-(J5-Pad11)
- U3 pad 8: /U3B7 -> (no net)
- U4 pad 19: /U4INTB -> (no net)
- U4 pad 20: /U4INTA -> (no net)
- U4 pad 27: Net-(J7-Pad9) -> Net-(J8-Pad11)
- U4 pad 28: /U4A7 -> (no net)
- U4 pad 7: Net-(J6-Pad9) -> Net-(J7-Pad11)
- U4 pad 8: /U4B7 -> (no net)
- U5 pad 19: /U5INTB -> (no net)
- U5 pad 20: /U5INTA -> (no net)
- U5 pad 27: Net-(J9-Pad9) -> Net-(J10-Pad11)
- U5 pad 28: /U5A7 -> (no net)
- U5 pad 7: Net-(J8-Pad9) -> Net-(J9-Pad11)
- U5 pad 8: /U5B7 -> (no net)
- U6 pad 24: /controller.sch/A1 -> /A1
- U6 pad 25: /controller.sch/A2 -> /A2
- U6 pad 26: /controller.sch/A3 -> /A3
Routing:
- net /U4A7: track 101.5 -> 0.00 mm, vias 2 -> 0
- net /U3A7: track 98.6 -> 0.00 mm, vias 2 -> 0
- net /U4INTA: track 86.1 -> 0.00 mm, vias 3 -> 0
- net /U4B7: track 78.0 -> 0.00 mm, vias 2 -> 0
- net /U3INTA: track 77.2 -> 0.00 mm, vias 1 -> 0
- net /U3INTB: track 73.7 -> 0.00 mm, vias 1 -> 0
- net /U3B7: track 72.7 -> 0.00 mm, vias 2 -> 0
- net /GND: track 80.0 -> 13.2 mm, vias 4 -> 0
- net /U4INTB: track 64.4 -> 0.00 mm, vias 2 -> 0
- net Net-(R2-Pad1): track 68.6 -> 6.60 mm, vias 3 -> 0
- net /controller.sch/A1: track 61.1 -> 0.00 mm
- net /A1: track 0.00 -> 61.0 mm
- net /controller.sch/A2: track 59.0 -> 0.00 mm
- net /A2: track 0.00 -> 58.8 mm
- net /controller.sch/A3: track 56.9 -> 0.00 mm
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Other:
- board text added: "C"
- board text added: "L+"
- board text added: "L-"
- board text removed: "COM"
- board text removed: "LED+"
- board text removed: "LED-"
- board text removed: "U3 A7"
- board text removed: "U3 B7"
- board text removed: "U3 INTA"
- board text removed: "U3 INTB"
- board text removed: "U4 A7"
- board text removed: "U4 B7"
- board text removed: "U4 INT B"
- board text removed: "U4 INTA"
- board text removed: "U5 A7"
- board text removed: "U5 B7"
- board text removed: "U5 INT B"
- board text removed: "U5 INTA"

Commit message: Some Tweaks I never pushed
Parts:
- moved U1 0.51 mm to (149.6, 116.8)
Routing:
- net /TXO: track 88.7 -> 88.0 mm
- net /BLE_DFU: track 28.0 -> 28.7 mm
- net /CTS: track 85.3 -> 84.8 mm
