File: Board-electronics/LED Board/LED Board.sch (KiCad schematic (older format))
At the start: 44 parts, among them J1 CONN_02X06, Q1 PN2222A, Q2 PN2222A, Q3 PN2222A

Commit message: more tweaking for perfection
Parts:
- R1, R10, R11, R12, R13, R14, R15, R16, R17, R18, R19, R2, R20, R3, R4, R5, R6, R7, R8, R9: footprint Resistors_THT:R_Axial_DIN0309_L9.0mm_D3.2mm_P12.70mm_Horizontal -> Resistors_THT:R_Axial_DIN0207_L6.3mm_D2.5mm_P10.16mm_Horizontal
Changed lines of the file:
@@
 F 0 "R1" V 2180 3100 50  0000 C CNN
 F 1 "R" V 2100 3100 50  0000 C CNN
-F 2 "Resistors_THT:R_Axial_DIN0309_L9.0mm_D3.2mm_P12.70mm_Horizontal" V 2030 3100 50  0001 C CNN
+F 2 "Resistors_THT:R_Axial_DIN0207_L6.3mm_D2.5mm_P10.16mm_Horizontal" V 2030 3100 50  0001 C CNN
 F 3 "" H 2100 3100 50  0001 C CNN
 	1    2100 3100
@@
 F 0 "R2" V 2530 3100 50  0000 C CNN
 F 1 "R" V 2450 3100 50  0000 C CNN
-F 2 "Resistors_THT:R_Axial_DIN0309_L9.0mm_D3.2mm_P12.70mm_Horizontal" V 2380 3100 50  0001 C CNN
+F 2 "Resistors_THT:R_Axial_DIN0207_L6.3mm_D2.5mm_P10.16mm_Horizontal" V 2380 3100 50  0001 C CNN
 F 3 "" H 2450 3100 50  0001 C CNN
 	1    2450 3100
@@
 F 0 "R3" V 2880 3100 50  0000 C CNN
 F 1 "R" V 2800 3100 50  0000 C CNN
-F 2 "Resistors_THT:R_Axial_DIN0309_L9.0mm_D3.2mm_P12.70mm_Horizontal" V 2730 3100 50  0001 C CNN
+F 2 "Resistors_THT:R_Axial_DIN0207_L6.3mm_D2.5mm_P10.16mm_Horizontal" V 2730 3100 50  0001 C CNN
 F 3 "" H 2800 3100 50  0001 C CNN
 	1    2800 3100
@@
 F 0 "R4" V 3230 3100 50  0000 C CNN
 F 1 "R" V 3150 3100 50  0000 C CNN
-F 2 "Resistors_THT:R_Axial_DIN0309_L9.0mm_D3.2mm_P12.70mm_Horizontal" V 3080 3100 50  0001 C CNN
+F 2 "Resistors_THT:R_Axial_DIN0207_L6.3mm_D2.5mm_P10.16mm_Horizontal" V 3080 3100 50  0001 C CNN
 F 3 "" H 3150 3100 50  0001 C CNN
 	1    3150 3100
@@
 F 0 "R5" V 3580 3100 50  0000 C CNN
 F 1 "R" V 3500 3100 50  0000 C CNN
-F 2 "Resistors_THT:R_Axial_DIN0309_L9.0mm_D3.2mm_P12.70mm_Horizontal" V 3430 3100 50  0001 C CNN
+F 2 "Resistors_THT:R_Axial_DIN0207_L6.3mm_D2.5mm_P10.16mm_Horizontal" V 3430 3100 50  0001 C CNN
 F 3 "" H 3500 3100 50  0001 C CNN
 	1    3500 3100
@@
 F 0 "R6" V 3930 3100 50  0000 C CNN
 F 1 "R" V 3850 3100 50  0000 C CNN
-F 2 "Resistors_THT:R_Axial_DIN0309_L9.0mm_D3.2mm_P12.70mm_Horizontal" V 3780 3100 50  0001 C CNN
+F 2 "Resistors_THT:R_Axial_DIN0207_L6.3mm_D2.5mm_P10.16mm_Horizontal" V 3780 3100 50  0001 C CNN
 F 3 "" H 3850 3100 50  0001 C CNN
 	1    3850 3100
@@
 F 0 "R7" V 4280 3100 50  0000 C CNN
 F 1 "R" V 4200 3100 50  0000 C CNN
-F 2 "Resistors_THT:R_Axial_DIN0309_L9.0mm_D3.2mm_P12.70mm_Horizontal" V 4130 3100 50  0001 C CNN
+F 2 "Resistors_THT:R_Axial_DIN0207_L6.3mm_D2.5mm_P10.16mm_Horizontal" V 4130 3100 50  0001 C CNN
 F 3 "" H 4200 3100 50  0001 C CNN
 	1    4200 3100
@@
 F 0 "R8" V 4980 3100 50  0000 C CNN
 F 1 "R" V 4900 3100 50  0000 C CNN
-F 2 "Resistors_THT:R_Axial_DIN0309_L9.0mm_D3.2mm_P12.70mm_Horizontal" V 4830 3100 50  0001 C CNN
+F 2 "Resistors_THT:R_Axial_DIN0207_L6.3mm_D2.5mm_P10.16mm_Horizontal" V 4830 3100 50  0001 C CNN
 F 3 "" H 4900 3100 50  0001 C CNN
 	1    4900 3100
@@
 F 0 "R9" V 5330 3100 50  0000 C CNN
 F 1 "R" V 5250 3100 50  0000 C CNN
-F 2 "Resistors_THT:R_Axial_DIN0309_L9.0mm_D3.2mm_P12.70mm_Horizontal" V 5180 3100 50  0001 C CNN
+F 2 "Resistors_THT:R_Axial_DIN0207_L6.3mm_D2.5mm_P10.16mm_Horizontal" V 5180 3100 50  0001 C CNN
 F 3 "" H 5250 3100 50  0001 C CNN
 	1    5250 3100
@@
 F 0 "R10" V 5680 3100 50  0000 C CNN
 F 1 "R" V 5600 3100 50  0000 C CNN
-F 2 "Resistors_THT:R_Axial_DIN0309_L9.0mm_D3.2mm_P12.70mm_Horizontal" V 5530 3100 50  0001 C CNN
+F 2 "Resistors_THT:R_Axial_DIN0207_L6.3mm_D2.5mm_P10.16mm_Horizontal" V 5530 3100 50  0001 C CNN
 F 3 "" H 5600 3100 50  0001 C CNN
 	1    5600 3100
@@
 F 0 "R11" V 6030 3100 50  0000 C CNN
 F 1 "R" V 5950 3100 50  0000 C CNN
-F 2 "Resistors_THT:R_Axial_DIN0309_L9.0mm_D3.2mm_P12.70mm_Horizontal" V 5880 3100 50  0001 C CNN
+F 2 "Resistors_THT:R_Axial_DIN0207_L6.3mm_D2.5mm_P10.16mm_Horizontal" V 5880 3100 50  0001 C CNN
 F 3 "" H 5950 3100 50  0001 C CNN
 	1    5950 3100
@@
 F 0 "R12" V 6380 3100 50  0000 C CNN
 F 1 "R" V 6300 3100 50  0000 C CNN
-F 2 "Resistors_THT:R_Axial_DIN0309_L9.0mm_D3.2mm_P12.70mm_Horizontal" V 6230 3100 50  0001 C CNN
+F 2 "Resistors_THT:R_Axial_DIN0207_L6.3mm_D2.5mm_P10.16mm_Horizontal" V 6230 3100 50  0001 C CNN
 F 3 "" H 6300 3100 50  0001 C CNN
 	1    6300 3100
@@
 F 0 "R13" V 6730 3100 50  0000 C CNN
 F 1 "R" V 6650 3100 50  0000 C CNN
-F 2 "Resistors_THT:R_Axial_DIN0309_L9.0mm_D3.2mm_P12.70mm_Horizontal" V 6580 3100 50  0001 C CNN
+F 2 "Resistors_THT:R_Axial_DIN0207_L6.3mm_D2.5mm_P10.16mm_Horizontal" V 6580 3100 50  0001 C CNN
 F 3 "" H 6650 3100 50  0001 C CNN
 	1    6650 3100
@@
 F 0 "R14" V 7080 3100 50  0000 C CNN
 F 1 "R" V 7000 3100 50  0000 C CNN
-F 2 "Resistors_THT:R_Axial_DIN0309_L9.0mm_D3.2mm_P12.70mm_Horizontal" V 6930 3100 50  0001 C CNN
+F 2 "Resistors_THT:R_Axial_DIN0207_L6.3mm_D2.5mm_P10.16mm_Horizontal" V 6930 3100 50  0001 C CNN
 F 3 "" H 7000 3100 50  0001 C CNN
 	1    7000 3100
@@
 F 0 "R15" V 7780 3100 50  0000 C CNN
 F 1 "R" V 7700 3100 50  0000 C CNN
-F 2 "Resistors_THT:R_Axial_DIN0309_L9.0mm_D3.2mm_P12.70mm_Horizontal" V 7630 3100 50  0001 C CNN
+F 2 "Resistors_THT:R_Axial_DIN0207_L6.3mm_D2.5mm_P10.16mm_Horizontal" V 7630 3100 50  0001 C CNN
 F 3 "" H 7700 3100 50  0001 C CNN
 	1    7700 3100
@@
 F 0 "R16" V 8130 3100 50  0000 C CNN
 F 1 "R" V 8050 3100 50  0000 C CNN
-F 2 "Resistors_THT:R_Axial_DIN0309_L9.0mm_D3.2mm_P12.70mm_Horizontal" V 7980 3100 50  0001 C CNN
+F 2 "Resistors_THT:R_Axial_DIN0207_L6.3mm_D2.5mm_P10.16mm_Horizontal" V 7980 3100 50  0001 C CNN
 F 3 "" H 8050 3100 50  0001 C CNN
 	1    8050 3100
@@
 F 0 "R17" V 8480 3100 50  0000 C CNN
 F 1 "R" V 8400 3100 50  0000 C CNN
-F 2 "Resistors_THT:R_Axial_DIN0309_L9.0mm_D3.2mm_P12.70mm_Horizontal" V 8330 3100 50  0001 C CNN
+F 2 "Resistors_THT:R_Axial_DIN0207_L6.3mm_D2.5mm_P10.16mm_Horizontal" V 8330 3100 50  0001 C CNN
 F 3 "" H 8400 3100 50  0001 C CNN
 	1    8400 3100
@@
 F 0 "R18" V 8880 3100 50  0000 C CNN
 F 1 "R" V 8800 3100 50  0000 C CNN
-F 2 "Resistors_THT:R_Axial_DIN0309_L9.0mm_D3.2mm_P12.70mm_Horizontal" V 8730 3100 50  0001 C CNN
+F 2 "Resistors_THT:R_Axial_DIN0207_L6.3mm_D2.5mm_P10.16mm_Horizontal" V 8730 3100 50  0001 C CNN
 F 3 "" H 8800 3100 50  0001 C CNN
 	1    8800 3100
@@
 F 0 "R19" V 9230 3100 50  0000 C CNN
 F 1 "R" V 9150 3100 50  0000 C CNN
-F 2 "Resistors_THT:R_Axial_DIN0309_L9.0mm_D3.2mm_P12.70mm_Horizontal" V 9080 3100 50  0001 C CNN
+F 2 "Resistors_THT:R_Axial_DIN0207_L6.3mm_D2.5mm_P10.16mm_Horizontal" V 9080 3100 50  0001 C CNN
 F 3 "" H 9150 3100 50  0001 C CNN
 	1    9150 3100
@@
 F 0 "R20" V 9580 3100 50  0000 C CNN
 F 1 "R" V 9500 3100 50  0000 C CNN
-F 2 "Resistors_THT:R_Axial_DIN0309_L9.0mm_D3.2mm_P12.70mm_Horizontal" V 9430 3100 50  0001 C CNN
+F 2 "Resistors_THT:R_Axial_DIN0207_L6.3mm_D2.5mm_P10.16mm_Horizontal" V 9430 3100 50  0001 C CNN
 F 3 "" H 9500 3100 50  0001 C CNN
 	1    9500 3100

Commit message: just some more tweaks
Parts:
- Q1, Q2, Q3: footprint TO_SOT_Packages_THT:TO-92_Molded_Narrow -> TO_SOT_Packages_THT:TO-92_Molded_Wide_Oval
Connections:
- net G: now also J1.11 (P11); no longer J1.9 (P9)
Changed lines of the file:
@@
 encoding utf-8
 Sheet 1 1
-Title ""
-Date ""
-Rev ""
-Comp ""
+Title "LED Display Board"
+Date "2017-05-16"
+Rev "1"
+Comp "Coppell School of Engineering"
 Comment1 ""
 Comment2 ""
@@
 F 0 "Q1" H 3450 1925 50  0000 L CNN
 F 1 "PN2222A" H 3450 1850 50  0000 L CNN
-F 2 "TO_SOT_Packages_THT:TO-92_Molded_Narrow" H 3450 1775 50  0001 L CIN
+F 2 "TO_SOT_Packages_THT:TO-92_Molded_Wide_Oval" H 3450 1775 50  0001 L CIN
 F 3 "" H 3250 1850 50  0001 L CNN
 	1    3250 1850
@@
 F 0 "Q2" H 6250 1925 50  0000 L CNN
 F 1 "PN2222A" H 6250 1850 50  0000 L CNN
-F 2 "TO_SOT_Packages_THT:TO-92_Molded_Narrow" H 6250 1775 50  0001 L CIN
+F 2 "TO_SOT_Packages_THT:TO-92_Molded_Wide_Oval" H 6250 1775 50  0001 L CIN
 F 3 "" H 6050 1850 50  0001 L CNN
 	1    6050 1850
@@
 F 0 "Q3" H 8900 1875 50  0000 L CNN
 F 1 "PN2222A" H 8900 1800 50  0000 L CNN
-F 2 "TO_SOT_Packages_THT:TO-92_Molded_Narrow" H 8900 1725 50  0001 L CIN
+F 2 "TO_SOT_Packages_THT:TO-92_Molded_Wide_Oval" H 8900 1725 50  0001 L CIN
 F 3 "" H 8700 1800 50  0001 L CNN
 	1    8700 1800
@@
 Text Label 5600 4400 0    60   ~ 0
 F
-Text Label 6400 4300 2    60   ~ 0
+Text Label 6400 4400 2    60   ~ 0
 G
 Wire Wire Line
-	6250 4300 6400 4300
-Wire Wire Line
 	5600 3900 5750 3900
 Wire Wire Line
@@
 Wire Wire Line
 	5600 4400 5750 4400
-NoConn ~ 6250 4400
 $Comp
 L LED D18
@@
 Text Notes 8850 3600 0    60   ~ 0
 Right Arrow\n
+Wire Wire Line
+	6400 4400 6250 4400
+NoConn ~ 6250 4300
 $EndSCHEMATC
